File: Schematics/TBHS-GPIO_Button_Matrix/controls_rev_3.brd (EAGLE design)
At the start: 108 x 50.8 mm, 40 parts

Commit message: Update schematic.
Connections:
- removed net N$10: D12.C, X.P$1, X.P$4
- new net N$5: D12.C, X.PIN0@0
- net 1: now also UP.PIN0@0; no longer UP.P$1, UP.P$4
- net N$11: now also C.PIN0@0; no longer C.P$1, C.P$4
- net N$12: now also LEFT.PIN0@0, LEFT.PIN0@1; no longer LEFT.P$1, LEFT.P$4
- net N$13: now also RIGHT.PIN0@0, RIGHT.PIN0@1; no longer RIGHT.P$1, RIGHT.P$4
- net N$14: now also DOWN.PIN0@0, DOWN.PIN0@1; no longer DOWN.P$1, DOWN.P$4
- net N$16: now also C-L.PIN0@0; no longer C-L.P$1, C-L.P$4
- net N$17: now also C-R.PIN0@0, C-R.PIN0@1; no longer C-R.P$1, C-R.P$4
- net N$2: now also SELECT.PIN0@0; no longer SELECT.P$1, SELECT.P$4
- net N$27: now also C-D.PIN0@0; no longer C-D.P$1, C-D.P$4
- net N$3: now also C-U.PIN0@0; no longer C-U.P$1, C-U.P$4
- net N$4: now also START.PIN0@0; no longer START.P$1, START.P$4
- net N$6: now also B.PIN0@0; no longer B.P$1, B.P$4
- net N$7: now also Z.PIN0@0; no longer Z.P$1, Z.P$4
- net N$8: now also Y.PIN0@0; no longer Y.P$1, Y.P$4
- net N$9: now also A.PIN0@0; no longer A.P$1, A.P$4
- net ROW_ONE: now also C-D.PIN1@1, C-L.PIN1@1, C-R.PIN1@1, C-U.PIN1@1; no longer C-D.P$2, C-D.P$3, C-L.P$2, C-L.P$3, C-R.P$2, C-R.P$3, C-U.P$2, C-U.P$3
- net ROW_THREE: now also B.PIN1@1, C.PIN1@1, Y.PIN1@1, Z.PIN1@1; no longer B.P$2, B.P$3, C.P$2, C.P$3, Y.P$2, Y.P$3, Z.P$2, Z.P$3
- net ROW_TWO: now also A.PIN1@1, SELECT.PIN1@1, START.PIN1@1, X.PIN1@1; no longer A.P$2, A.P$3, SELECT.P$2, SELECT.P$3, START.P$2, START.P$3, X.P$2, X.P$3
- net ROW_ZERO: now also DOWN.PIN1@1, LEFT.PIN1@1, RIGHT.PIN1@1, UP.PIN1@1; no longer DOWN.P$2, DOWN.P$3, LEFT.P$2, LEFT.P$3, RIGHT.P$2, RIGHT.P$3, UP.P$2, UP.P$3
Routing:
- net ROW_ONE: track 78.4 -> 66.6 mm
- net ROW_TWO: track 50.1 -> 39.8 mm
- net ROW_ZERO: track 23.9 -> 16.1 mm
- net N$4: track 7.51 -> 0.00 mm
- net N$9: track 4.79 -> 0.00 mm
- net N$7: track 3.91 -> 0.00 mm
- net ROW_THREE: track 62.8 -> 59.2 mm
- net N$5: track 0.00 -> 3.53 mm
- net N$10: track 3.53 -> 0.00 mm
- net N$16: track 3.12 -> 0.00 mm
